File: Nitin/PCB/Kitty_PCB.sch (EAGLE design)
At the start: 49 parts

Commit message: PCB 1.0 Final
1st version of the PCB is completed.
Parts:
- removed C1: (no value), robocon:CAPACITOR050-075X075
- removed LED2, LED3: LED, robocon:LED
- removed R3: (no value), robocon:RESISTANCE0207/10
- added 9VLED: LED, robocon:LED
- renumbered LED1 to 5VLED, LED4 to A1LED, LED5 to A2LED
Connections:
- removed net N$115: LED3.C, R3.1
- new net N$8: A2LED.A, R5.2
- net 12V_OUT: no longer C1.1, LED3.A
- net GND: now also 9VLED.C; no longer A2LED.A, C1.2, LED2.C, R3.2, R5.2
- net N$19: now also 9VLED.A; no longer LED2.A
