File: Nitin/PCB - Copy/Kitty_PCB.brd (EAGLE design)
At the start: 204.4 x 284.1 mm, 46 parts

Commit message: PCB 1.0 Final
1st version of the PCB is completed.
Parts:
- added 12VLED: LED, robocon:LED3MM
- added C1: (no value), robocon:C050-075X075
- added R3: (no value), robocon:0207/10
- moved 7809B 19.0 mm to (45.7, -95.2)
- moved 7809 16.5 mm to (26.7, -95.2)
- moved MOSFET 3.59 mm to (44.5, -16.5)
Connections:
- new net N$115: 12VLED.K, R3.1
- net 12V_OUT: now also 12VLED.A, C1.1
- net GND: now also C1.2, R3.2
Routing:
- net GND: track 346.0 -> 976.4 mm
- net 9V: track 478.6 -> 0.00 mm, vias 2 -> 0
- net 5V: track 795.0 -> 568.6 mm, vias 1 -> 0
- net A1SC2: track 245.8 -> 139.4 mm
- net 25A2: track 197.4 -> 136.8 mm, vias 0 -> 1
- net 25A1: track 180.0 -> 237.3 mm, vias 1 -> 0
- net 27A1: track 189.7 -> 136.0 mm
- net 23A2: track 204.0 -> 153.9 mm, vias 0 -> 1
- net 12V_OUT: track 199.7 -> 162.4 mm
- net 7A1: track 111.5 -> 145.2 mm
- net 19A1: track 132.9 -> 160.8 mm, vias 1 -> 0
- net A1SC1: track 149.6 -> 121.8 mm
- net A2SC1: track 130.8 -> 103.9 mm
- net 5A1: track 165.8 -> 139.4 mm, vias 0 -> 1
- net 21A1: track 80.0 -> 105.6 mm
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- removed copper zone on layer 1, net GND
- removed copper zone on layer 16, net GND
