File: Nitin/PCB/PCB_Final/Kitty_PCB.brd (EAGLE design)
At the start: 204.4 x 284.1 mm, 49 parts

Commit message: PCB1 Final
Final PCB for ettching completed.
Parts:
- removed 12VLED: LED, robocon:LED3MM
- removed C1: (no value), robocon:C050-075X075
- removed R3: (no value), robocon:0207/10
- moved A1LED 31.9 mm to (56.1, -234.9)
- moved U$1 21.7 mm to (55.9, -130.8)
- moved R4 14.0 mm to (61.2, -227.3)
- moved SCREW_TERMINAL2 10.9 mm to (25.4, -8.89)
- moved SCREW_TERMINAL_1 9.25 mm to (40.6, -8.89)
- moved R2 8.98 mm to (57.1, -61.0), turned to 90 degrees
- moved 7809B 8.98 mm to (36.8, -94.0)
- moved MOSFET 5.68 mm to (41.9, -21.6)
- moved ENCODER1 5.08 mm to (182.9, -219.7)
- moved ENCODER2 5.08 mm to (182.9, -176.5)
- moved ENCODER7 5.08 mm to (182.9, -73.7)
- moved ENCODER8 5.08 mm to (182.9, -35.6)
- moved 7809 1.80 mm to (27.9, -94.0)
- moved 5VLED 1.27 mm to (26.7, -162.6)
Connections:
- removed net N$115: 12VLED.K, R3.1
- net 12V_OUT: no longer 12VLED.A, C1.1
- net GND: no longer C1.2, R3.2
Routing:
- net GND: track 892.7 -> 380.9 mm, vias 2 -> 18
- net 9V: track 0.00 -> 454.4 mm, vias 0 -> 2
- net 5V: track 580.2 -> 761.6 mm, vias 0 -> 3
- net 23A2: track 131.0 -> 204.0 mm, vias 1 -> 0
- net A1SC2: track 170.3 -> 239.1 mm, vias 1 -> 0
- net 25A2: track 136.8 -> 193.9 mm, vias 1 -> 0
- net 27A1: track 140.7 -> 181.9 mm
- net 5A1: track 124.6 -> 164.3 mm
- net 25A1: track 208.2 -> 180.0 mm, vias 0 -> 1
- net 21A1: track 105.6 -> 77.8 mm
- net A2SC1: track 103.9 -> 130.8 mm
- net 19A2: track 138.6 -> 115.8 mm
- net 7A1: track 130.3 -> 111.5 mm, vias 1 -> 0
- net 27A2: track 185.3 -> 167.8 mm
- net 29A2: track 194.1 -> 177.2 mm
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- added copper zone on layer 1, net GND
- added copper zone on layer 16, net GND
Other:
- board size 204.4 x 284.1 mm -> 193 x 279.1 mm
- board text added: "9V"
- board text added: "E6"
- board text added: "KITTY1.0"
- board text removed: "KITTY V1"
