File: Nitin/PCB/PCB_Final/Kitty_PCB.sch (EAGLE design)
At the start: 49 parts

Commit message: PCB1 Final
Final PCB for ettching completed.
Parts:
- removed 12VLED: LED, robocon:LED
- removed C1: (no value), robocon:CAPACITOR050-075X075
- removed R3: (no value), robocon:RESISTANCE0207/10
Connections:
- removed net N$115: 12VLED.C, R3.1
- net 12V_OUT: no longer 12VLED.A, C1.1
- net GND: no longer C1.2, R3.2
Changed lines of the file:
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@@
 <clearance class="0" value="0.8128"/>
-</class>
-<class number="1" name="GND" width="0" drill="0">
-</class>
-<class number="2" name="9V" width="2.54" drill="2.54">
-<clearance class="2" value="0.8128"/>
-</class>
-<class number="3" name="12V" width="3.556" drill="3.556">
-<clearance class="3" value="0.8128"/>
-</class>
-<class number="4" name="5V" width="1.778" drill="1.778">
-<clearance class="4" value="0.8128"/>
 </class>
 </classes>
@@
 <part name="SV15" library="robocon" deviceset="RELIMATE_03-1" device=""/>
 <part name="SV16" library="robocon" deviceset="RELIMATE_03-1" device=""/>
-<part name="12VLED" library="robocon" deviceset="LED" device=""/>
-<part name="C1" library="robocon" deviceset="CAPACITOR" device="050-075X075"/>
-<part name="R3" library="robocon" deviceset="RESISTANCE" device="0207/10"/>
 <part name="ENCODER1" library="robocon" deviceset="RELIMATE_05-1" device=""/>
 <part name="ENCODER2" library="robocon" deviceset="RELIMATE_05-1" device=""/>
@@
 <attribute name="NAME" x="-379.73" y="69.342" size="1.778" layer="95"/>
 </instance>
-<instance part="12VLED" gate="G$1" x="-109.22" y="-7.62" smashed="yes">
-<attribute name="NAME" x="-105.664" y="-12.192" size="1.778" layer="95" rot="R90"/>
-</instance>
-<instance part="C1" gate="G$1" x="-111.76" y="-33.02" smashed="yes">
-<attribute name="NAME" x="-110.236" y="-32.639" size="1.778" layer="95"/>
-<attribute name="VALUE" x="-110.236" y="-37.719" size="1.778" layer="96"/>
-</instance>
-<instance part="R3" gate="G$1" x="-96.52" y="-17.78" smashed="yes">
-<attribute name="NAME" x="-100.33" y="-16.2814" size="1.778" layer="95"/>
-<attribute name="VALUE" x="-100.33" y="-21.082" size="1.778" layer="96"/>
-</instance>
 <instance part="ENCODER1" gate="G$1" x="-444.5" y="-5.08" smashed="yes">
 <attribute name="VALUE" x="-445.77" y="-15.24" size="1.778" layer="96"/>
@@
 </segment>
 <segment>
-<pinref part="C1" gate="G$1" pin="2"/>
-<junction x="-111.76" y="-38.1"/>
-<label x="-109.22" y="-38.1" size="1.778" layer="95"/>
-</segment>
-<segment>
-<pinref part="R3" gate="G$1" pin="2"/>
-<junction x="-91.44" y="-17.78"/>
-<label x="-91.44" y="-17.78" size="1.778" layer="95"/>
-</segment>
-<segment>
 <pinref part="ENCODER1" gate="G$1" pin="2"/>
 <junction x="-436.88" y="-7.62"/>
@@
 </segment>
 </net>
-<net name="5V" class="4">
+<net name="5V" class="0">
 <segment>
 <pinref part="U$1" gate="G$1" pin="OUT+"/>
@@
 </segment>
 </net>
-<net name="12V_OUT" class="3">
+<net name="12V_OUT" class="0">
 <segment>
 <pinref part="MOSFET" gate="1" pin="IN"/>
@@
 </segment>
 <segment>
-<pinref part="12VLED" gate="G$1" pin="A"/>
-<wire x1="-109.22" y1="-5.08" x2="-121.92" y2="-5.08" width="0.1524" layer="91"/>
-<wire x1="-121.92" y1="-5.08" x2="-121.92" y2="-30.48" width="0.1524" layer="91"/>
-<pinref part="C1" gate="G$1" pin="1"/>
-<wire x1="-121.92" y1="-30.48" x2="-111.76" y2="-30.48" width="0.1524" layer="91"/>
-<label x="-109.22" y="-5.08" size="1.778" layer="95"/>
-</segment>
-<segment>
 <pinref part="7809" gate="1" pin="IN"/>
 <junction x="-223.52" y="99.06"/>
@@
 </segment>
 </net>
-<net name="12V_IN_GND" class="3">
+<net name="12V_IN_GND" class="0">
 <segment>
 <pinref part="MOSFET" gate="1" pin="GND"/>
@@
 </segment>
 </net>
-<net name="9V" class="2">
+<net name="9V" class="0">
 <segment>
 <pinref part="7809" gate="1" pin="OUT"/>
@@
 </segment>
 </net>
-<net name="N$115" class="0">
-<segment>
-<pinref part="12VLED" gate="G$1" pin="C"/>
-<pinref part="R3" gate="G$1" pin="1"/>
-<wire x1="-109.22" y1="-12.7" x2="-109.22" y2="-17.78" width="0.1524" layer="91"/>
-<wire x1="-109.22" y1="-17.78" x2="-101.6" y2="-17.78" width="0.1524" layer="91"/>
-</segment>
-</net>
